Commit message: Change camera to RGBD

File: meine_bot/urdf/meine_bot.xacro (robot description, xacro)
@@ -63,5 +63,5 @@
   <xacro:wheel_default name="left" reflect="1"/>
   <xacro:wheel_default name="right" reflect="-1"/>
-  <link name="camera">
+  <link name="camera_link">
     <inertial>
       <mass value ="0.1"/>
@@ -90,7 +90,7 @@
   </link>
   <joint name="camera_joint" type="fixed">
-    <origin xyz="${length/2} 0 ${-camera_height /2}" rpy="0 0 0"/>
+    <origin xyz="${length/2} 0 ${-camera_height /2}" rpy="${pi/2} 0 0"/>
     <parent link="chassis"/>
-    <child link="camera" />
+    <child link="camera_link" />
   </joint>
   <link name="hokuyo">

File: meine_bot/urdf/meine_bot_values.xacro (robot description, xacro)
@@ -20,7 +20,7 @@
   <xacro:property name="battery_mass" value="5"/>
   <!-- CAMERA -->
-  <xacro:property name="camera_width" value="0.03"/>
-  <xacro:property name="camera_length" value="0.03"/>
-  <xacro:property name="camera_height" value="0.02"/>
+  <xacro:property name="camera_width" value=".005"/>
+  <xacro:property name="camera_length" value="0.05"/>
+  <xacro:property name="camera_height" value="0.05"/>
   <!-- HOKUYO -->
   <xacro:property name="hokuyo_width" value="0.1"/>

Commit message: Rotate the camera joint in 90 degrees

File: meine_bot/urdf/meine_bot.xacro (robot description, xacro)
@@ -90,5 +90,5 @@
   </link>
   <joint name="camera_joint" type="fixed">
-    <origin xyz="${length/2} 0 ${-camera_height /2}" rpy="${pi/2} 0 0"/>
+    <origin xyz="${length/2} 0 ${-camera_height /2}" rpy="0 0 0"/>
     <parent link="chassis"/>
     <child link="camera_link" />

Commit message: Add RGBD camera frame

File: meine_bot/urdf/meine_bot.xacro (robot description, xacro)
@@ -94,4 +94,10 @@
     <child link="camera_link" />
   </joint>
+  <link name="camera_rgbd_frame"></link>
+  <joint name="camera_rgbd_frame" type="fixed">
+    <origin rpy="0 0 0"/>
+    <parent link="camera_link"/>
+    <child link="camera_rgbd_frame"/>
+  </joint>
   <link name="hokuyo">
     <inertial>

Commit message: Fix Topics names

File: meine_bot/urdf/meine_bot.xacro (robot description, xacro)
@@ -95,5 +95,5 @@
   </joint>
   <link name="camera_rgbd_frame"></link>
-  <joint name="camera_rgbd_frame" type="fixed">
+  <joint name="camera_rgbd_joint" type="fixed">
     <origin rpy="0 0 0"/>
     <parent link="camera_link"/>

Commit message: Rotate rgbd frame

File: meine_bot/urdf/meine_bot.xacro (robot description, xacro)
@@ -96,5 +96,5 @@
   <link name="camera_rgbd_frame"></link>
   <joint name="camera_rgbd_joint" type="fixed">
-    <origin rpy="0 0 0"/>
+    <origin rpy="${-pi/2} 0 ${-pi/2}"/>
     <parent link="camera_link"/>
     <child link="camera_rgbd_frame"/>
